File: pcb/BreadBoard-Power.kicad_sch (KiCad schematic)
At the start: 14 parts, among them J1 USB_C, J2 Rail1, J3 Rail2, U1 AMS1117-3.3

Commit message: docs: schematic cleanup
Connections:
- net D2: now reaches D2.1 (K), R4.1
- net D1: now reaches D1.1 (K), R3.1
Changed lines of the file:
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@@
 	(generator_version "8.0")
 	(paper "A4")
-    (title_block
-                (title "BreadBoard-Power")
-                (date "${DATE}")
-                (rev "${VERSION}")
-                (company "Qetesh")
-            )
+	(title_block
+		(title "BreadBoard-Power")
+		(date "${DATE}")
+		(rev "${VERSION}")
+		(company "Qetesh")
+	)
 	(junction
 		(at 142.24 58.42)
@@
 	)
 	(junction
-		(at 124.46 49.53)
-		(diameter 0)
-		(color 0 0 0 0)
-	)
-	(junction
 		(at 90.17 55.88)
 		(diameter 0)
@@
 	)
 	(junction
-		(at 153.67 49.53)
-		(diameter 0)
-		(color 0 0 0 0)
-	)
-	(junction
 		(at 50.8 73.66)
 		(diameter 0)
@@
 	(wire
 		(pts
-			(xy 124.46 48.26) (xy 124.46 49.53)
-		)
-		(stroke
-			(width 0)
-			(type default)
-		)
-	)
-	(wire
-		(pts
 			(xy 168.91 55.88) (xy 171.45 55.88)
 		)
@@
 		(pts
 			(xy 156.21 58.42) (xy 153.67 58.42)
-		)
-		(stroke
-			(width 0)
-			(type default)
-		)
-	)
-	(wire
-		(pts
-			(xy 153.67 48.26) (xy 153.67 49.53)
 		)
 		(stroke
@@
 		)
 	)
+	(label "D1"
+		(at 184.15 53.34 0)
+		(fields_autoplaced yes)
+		(effects
+			(font
+				(size 1.27 1.27)
+			)
+			(justify left bottom)
+		)
+	)
 	(label "Rail1"
 		(at 124.46 54.61 90)
@@
 		(fields_autoplaced yes)
 		(effects
+			(font
+				(size 1.27 1.27)
+			)
+			(justify left bottom)
+		)
+	)
+	(label "D2"
+		(at 193.04 53.34 0)
+		(fields_autoplaced yes)
+		(effects
