File: pcb/BreadBoard-Power.kicad_pcb (KiCad board)
At the start: 2 copper layers, 10.5 x 61 mm, 14 parts, among them J1 USB_C, J2 Rail1, J3 Rail2, U1 AMS1117-3.3

Commit message: docs: schematic cleanup
Connections:
- net Net-(D1-K) renamed /D1
- net Net-(D2-K) renamed /D2
Changed lines of the file:
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@@
 	(net 6 "/Rail1")
 	(net 7 "/Rail2")
-	(net 8 "Net-(D1-K)")
-	(net 9 "Net-(D2-K)")
+	(net 8 "/D1")
+	(net 9 "/D2")
 	(footprint "LED_SMD:LED_0603_1608Metric_Pad1.05x0.95mm_HandSolder"
 		(layer "F.Cu")
@@
 			(layers "F.Cu" "F.Paste" "F.Mask")
 			(roundrect_rratio 0.25)
-			(net 9 "Net-(D2-K)")
+			(net 9 "/D2")
 			(pinfunction "K")
 			(pintype "passive")
@@
 			(layers "F.Cu" "F.Paste" "F.Mask")
 			(roundrect_rratio 0.25)
-			(net 8 "Net-(D1-K)")
+			(net 8 "/D1")
 			(pintype "passive")
 		)
@@
 			(layers "F.Cu" "F.Paste" "F.Mask")
 			(roundrect_rratio 0.25)
-			(net 8 "Net-(D1-K)")
+			(net 8 "/D1")
 			(pinfunction "K")
 			(pintype "passive")
@@
 			(layers "F.Cu" "F.Paste" "F.Mask")
 			(roundrect_rratio 0.25)
-			(net 9 "Net-(D2-K)")
-			(pintype "passive")
-		)
+			(net 9 "/D2")
+			(pintype "passive")
+		)

Commit message: fix: add missing logos
Parts:
- added G***: LOGO, My_Footprints:CutieMark5mmInverted, B.Cu at (190.0, 58.5)
- added G***: LOGO, My_Footprints:qr_qete.sh-el_08, B.Cu at (190.0, 98.2)
- added REF**: OSHW-Logo_5.7x6mm_SilkScreen, Symbol:OSHW-Logo_5.7x6mm_SilkScreen, B.Cu at (190.0, 77.0)

Commit message: feat: add production rails
Parts:
- added REF**: JLCPCB_Tooling_Hole, My_Footprints:JLCPCB_Tooling_Hole, F.Cu at (186.2, 37.8)
- added REF**: JLCPCB_Tooling_Hole, My_Footprints:JLCPCB_Tooling_Hole, F.Cu at (193.8, 37.8)
- added REF**: JLCPCB_Tooling_Hole, My_Footprints:JLCPCB_Tooling_Hole, F.Cu at (186.2, 108.8)
- added REF**: JLCPCB_Tooling_Hole, My_Footprints:JLCPCB_Tooling_Hole, F.Cu at (193.8, 108.8)
- added mouse-bite-2mm-slot: VAL**, Panelization:mouse-bite-2x5mm-slot-onesided-v2, F.Cu at (190.0, 104.2)
- added mouse-bite-2mm-slot: VAL**, Panelization:mouse-bite-2x5mm-slot-onesided-no-edge, F.Cu at (190.0, 41.2)
Other:
- board size 10.5 x 61 mm -> 10.5 x 74 mm
